File: Hardware/PCB/IoT_Board/IoT_Board.kicad_sch (KiCad schematic)
At the start: 113 parts, among them J1 KF7.62-2P, J10 Conn_01x02_Pin, J6 Conn_01x04_Pin, J7 Conn_01x04_Pin, J8 Conn_01x04_Pin, J9 Conn_01x04_Pin, K1 SRD-12VDC-SL-C, K2 SRD-12VDC-SL-C, K3 SRD-12VDC-SL-C, Q2 AO3400A, Q3 AO3400A, Q4 AO3400A, T1 ZMPT101B, U1 ESP32-S3-WROOM-1, U14 ADS1256IDBR, U15 MCP6002-xSN, U16 MCP6002-xSN, U18 MCP6002-xSN, U19 MCP6002-xSN, U2 LM385S-2.5, U20 AMS1117-3.3, U22 AMS1117-3.3, U4 HLK-5M05, U5 PC817, U6 PC817, U7 PC817, Y2 8MHz

Commit message: done sche
Parts:
- removed C29, C30: 22pF, Resistor_SMD:R_0805_2012Metric_Pad1.20x1.40mm_HandSolder, symbol Device:C
- removed C31, C45, C55: 10uF, Resistor_SMD:R_0805_2012Metric_Pad1.20x1.40mm_HandSolder, symbol Device:C
- removed C34, C35, C36, C37, C38, C39, C40, C41, C42, C43, C44, C46, C47, C48, C49, C50, C53: 100nF, Resistor_SMD:R_0805_2012Metric_Pad1.20x1.40mm_HandSolder, symbol Device:C
- removed C54: 1uF, Resistor_SMD:R_0805_2012Metric_Pad1.20x1.40mm_HandSolder, symbol Device:C
- removed J6, J7, J8, J9: Conn_01x04_Pin, Connector_PinHeader_2.54mm:PinHeader_1x04_P2.54mm_Vertical, symbol Connector:Conn_01x04_Pin
- removed NT2: NetTie_2, NetTie:NetTie-2_THT_Pad0.3mm, symbol Device:NetTie_2
- removed PS1: B0505S-2W, B050S:B0505S2W, symbol B050s-2W:B0505S-2W
- removed R45, R46, R51, R66, R67, R68, R69, R70, R71: 10K, Resistor_SMD:R_0805_2012Metric_Pad1.20x1.40mm_HandSolder, symbol Device:R
- removed R47, R48, R49, R50: 100R, Resistor_SMD:R_0805_2012Metric_Pad1.20x1.40mm_HandSolder, symbol Device:R
- removed T1: ZMPT101B, ZMPT101B:XFMR_ZMPT101B, symbol My Sym:ZMPT101B
- removed U14: ADS1256IDBR, ADS:SOP65P780X200-28N, symbol ADS1256:ADS1256IDBR
- removed U15, U16, U18, U19: MCP6002-xSN, MCP6002:SOIC8-N_MC_MCH-M, symbol Amplifier_Operational:MCP6002-xSN
- removed U2: LM385S-2.5, Package_SO:SOIC-8_3.9x4.9mm_P1.27mm, symbol Reference_Voltage:LM385S-2.5
- removed U20: AMS1117-3.3, Package_TO_SOT_SMD:SOT-223-3_TabPin2, symbol Regulator_Linear:AMS1117-3.3
- removed Y2: 8MHz, Crystal:Resonator-2Pin_W7.0mm_H2.5mm, symbol Device:Crystal
- added BL1, BL2, BL3: (no value), Package_SO:SSOP-10_3.9x4.9mm_P1.00mm, symbol Sym:BL0942
- added C59, C67, C73, C76: 100uF, Resistor_SMD:R_0805_2012Metric_Pad1.20x1.40mm_HandSolder, symbol Device:C
- added C66: 1uF, Resistor_SMD:R_0805_2012Metric_Pad1.20x1.40mm_HandSolder, symbol Device:C
- added C69, C70, C71, C72, C74, C75, C77: 33nF, Resistor_SMD:R_0805_2012Metric_Pad1.20x1.40mm_HandSolder, symbol Device:C
- added D1: IR204A, LED_THT:LED_D3.0mm_IRBlack, symbol LED:IR204A
- added D33, D34, D35, D36, D38: LED, LED_SMD:LED_0805_2012Metric_Pad1.15x1.40mm_HandSolder, symbol Device:LED
- added IC1: VS1838B, Footprint:VS1838B, symbol Sym:VS1838B
- added J11, J12, J13: KF7.62-2P, KF7.62:2P, symbol KF-7.62:KF7.62-2P
- added J14: MAX_98357, Connector_PinHeader_1.00mm:PinHeader_1x07_P1.00mm_Vertical, symbol Connector:Conn_01x07_Pin
- added J15: INMP_441, Connector_PinHeader_2.54mm:PinHeader_2x03_P2.54mm_Vertical, symbol Connector_Generic:Conn_02x03_Counter_Clockwise
- added J2: Debug UART0, Connector_JST:JST_XH_B4B-XH-A_1x04_P2.50mm_Vertical, symbol Connector:Conn_01x04_Pin
- added J4: UART1, Connector_JST:JST_XH_B4B-XH-A_1x04_P2.50mm_Vertical, symbol Connector:Conn_01x04_Pin
- added J5: I2C, Connector_JST:JST_XH_B4B-XH-A_1x04_P2.50mm_Vertical, symbol Connector:Conn_01x04_Pin
- added J6, J7, J8: CT, Connector_JST:JST_XH_B2B-XH-A_1x02_P2.50mm_Vertical, symbol Connector:Conn_01x02_Pin
- added J9: USB_C_Receptacle_USB2.0_16P, Connector_USB:USB_C_Receptacle_HCTL_HC-TYPE-C-16P-01A, symbol Connector:USB_C_Receptacle_USB2.0_16P
- added Q1: AO3400A, Package_TO_SOT_SMD:SOT-23, symbol Transistor_FET:AO3400A
- added R34, R35: 4k7, Resistor_SMD:R_0805_2012Metric_Pad1.20x1.40mm_HandSolder, symbol Device:R
- added R36, R39: 100R, Resistor_SMD:R_0805_2012Metric_Pad1.20x1.40mm_HandSolder, symbol Device:R
- added R37: 10K, Resistor_SMD:R_0805_2012Metric_Pad1.20x1.40mm_HandSolder, symbol Device:R
- added R38: 33R, Resistor_SMD:R_0805_2012Metric_Pad1.20x1.40mm_HandSolder, symbol Device:R
- added R40, R42, R43, R44, R72: 4K7, Resistor_SMD:R_0805_2012Metric_Pad1.20x1.40mm_HandSolder, symbol Device:R
- added R41: 0R, Resistor_SMD:R_0805_2012Metric_Pad1.20x1.40mm_HandSolder, symbol Device:R
- added R45, R46: 5.1k, Resistor_SMD:R_0805_2012Metric, symbol Device:R_Small
- added R78, R81, R83: 220R, Resistor_SMD:R_0805_2012Metric_Pad1.20x1.40mm_HandSolder, symbol Device:R
- added R79, R80: 1K, Resistor_SMD:R_0805_2012Metric_Pad1.20x1.40mm_HandSolder, symbol Device:R
- added SW1, SW2, SW3, SW4: SW_Push, Button_Switch_SMD:SW_Tactile_SPST_NO_Straight_CK_PTS636Sx25SMTRLFS, symbol Switch:SW_Push
- added TR1: ZMPT101K, Transformer_THT:Transformer_Zeming_ZMPT101K, symbol Transformer:ZMPT101K
- C52, C58: value 100nF -> 10uF
- C56: value 10uF -> 100uF
- C61, C62: value 100nF -> 1uF
- C64: value 10uF -> 1uF
- K1, K2, K3: footprint RL10SRD:RELAY_SRD-12VDC-SL-C -> Footprint:RELAY_SRD-12VDC-SL-C
- R52, R55, R58: value 10K -> 33R
- R53, R54, R56, R57: value 10K -> 1K
- R59, R60: value 100R -> 1K
- R61: value 100R -> 100K
- R62: value 100R -> 33R
- R63: value 10K -> 100K
- R64: value 10K -> 0R
- R65: value 1K -> 0R
- U5, U6, U7: footprint PC817_SMD:DIL04 -> Footprint:SOP254P960X420-4N
Connections:
- net GND1 is gone; now on net GND: J10.2 (Pin_2), Q2.2 (S), Q3.2 (S), Q4.2 (S), R29.1, R30.1, R31.1, U4.3 (-Vout)
- net PC13 is gone; now on net LED1: R77.2
- net +3V3: now also R64.2, R65.2, U1.2 (3V3), BL1.1 (VDD), BL2.1 (VDD), BL3.1 (VDD), C59.1, C67.2, C73.2, C76.2, D33.2 (A), D34.2 (A), D35.2 (A), D38.2 (A), J15.5 (Pin_5), J5.1 (Pin_1), R34.2, R35.2, R36.2, R37.2, R42.1, R43.1, R44.1, R72.1; no longer C61.2, C62.2, C64.2
- net +5V: now also C52.2, C56.1, C57.2, C58.2, U22.3 (VI), D36.2 (A), J14.7 (Pin_7), J9.A4 (VBUS), J9.A9 (VBUS), J9.B4 (VBUS), J9.B9 (VBUS), R38.1
- net COM1: now also J11.2; no longer K2.COM, K3.COM, R3.1, R4.1
- net O1: now also J11.1; no longer C2.2, C3.2, K2.NO, K3.NO
- net RL1: now also U1.4 (IO4); no longer U6.2, U7.2
- net at R56.1: now also R55.1, J7.1 (Pin_1); no longer R58.2
- net GND: now reaches R60.1
- net GND: now also C51.2, C52.1, C56.2, C57.1, C58.1, C60.1, C61.1, C62.1, C63.1, C64.1, C65.1, R52.2, R54.1, R55.2, R57.1, R58.2, R62.1, U1.1 (GND), U1.40 (GND), U1.41 (GND), U22.1 (GND), BL1.5 (GND), BL1.7 (SEL), BL1.8 (SCLK_BPS), BL2.5 (GND), BL2.7 (SEL), BL2.8 (SCLK_BPS), BL3.5 (GND), BL3.7 (SEL), BL3.8 (SCLK_BPS), C59.2, C66.1, C67.1, C69.2, C70.1, C71.1, C72.2, C73.1, C74.1, C75.2, C76.1, C77.2, IC1.2 (GND), J14.6 (Pin_6), J15.1 (Pin_1), J15.6 (Pin_6), J2.4 (Pin_4), J4.4 (Pin_4), J5.4 (Pin_4), J6.2 (Pin_2), J7.2 (Pin_2), J8.2 (Pin_2), J9.A1 (GND), J9.A12 (GND), J9.B1 (GND), J9.B12 (GND), J9.SH (SHIELD), Q1.2 (S), R40.2, R41.1, R45.2, R46.2, R81.2, R83.2, SW1.2, SW2.2, SW3.2, SW4.2, TR1.3
- net at R61.2: now also R63.1
- net L: now reaches R61.1
- net L: now also J1.2, U4.1 (AC/L); no longer R64.2
- net at R59.1: now also R58.1, J8.1 (Pin_1); no longer R63.2
- net at R59.2: now also BL3.2 (IP), C74.2
- net at R60.2: now also BL3.3 (IN), C75.1
- net at R57.2: now also BL2.3 (IN), C72.1; no longer R55.1
- net N: now reaches J1.1, U4.2 (AC/N)
- net N: now also TR1.2
- net at R53.1: now also R52.1, J6.1 (Pin_1)
- net VP: now reaches R62.2
- net VP: now also BL1.4 (VP), BL2.4 (VP), BL3.4 (VP), C77.1, TR1.4
- net SP_BCLK: now reaches U1.10 (IO17)
- net SP_BCLK: now also J14.2 (Pin_2)
- net SP_LRC: now reaches U1.11 (IO18)
- net SP_LRC: now also J14.1 (Pin_1)
- net MIC_DIN: now reaches U1.12 (IO8)
- net MIC_DIN: now also J15.4 (Pin_4)
- net USB_D-: now reaches U1.13 (USB_D-)
- net USB_D-: now also J9.A7 (D-), J9.B7 (D-)
- net USB_D+: now reaches U1.14 (USB_D+)
- net USB_D+: now also J9.A6 (D+), J9.B6 (D+)
- net BUT2: now reaches U1.15 (IO3)
- net BUT2: now also C66.2, R72.2, SW4.1
- net BL_TX: now reaches U1.17 (IO9)
- net BL_TX: now also BL1.9 (RX), BL2.9 (RX), BL3.9 (RX)
- net BL_RX1: now reaches U1.18 (IO10)
- net BL_RX1: now also BL1.10 (TX), BL2.10 (TX), BL3.10 (TX)
- net BL_RX2: now reaches U1.19 (IO11)
- net BL_RX2: now also BL2.6 (CF1)
- net BL_RX3: now reaches U1.20 (IO12)
- net BL_RX3: now also BL3.6 (CF1)
- net SP_DOUT: now reaches U1.23 (IO21)
- net SP_DOUT: now also J14.3 (Pin_3)
- net LED2: now reaches U1.24 (IO47)
- net LED2: now also R78.2
- net LED1: now reaches U1.25 (IO48)
- net BOOT: now reaches U1.27 (IO0)
- net BOOT: now also C62.2, R43.2, SW2.1
- net EN: now reaches U1.3 (EN)
- net EN: now also C61.2, R42.2, SW1.1
- net TX1: now reaches U1.31 (IO38)
- net TX1: now also J4.2 (Pin_2)
- net RX1: now reaches U1.32 (IO39)
- net RX1: now also J4.3 (Pin_3)
- net IR_TX: now reaches U1.33 (IO40)
- net IR_TX: now also R39.1
- net I2C_SDA: now reaches U1.34 (IO41)
- net I2C_SDA: now also J5.2 (Pin_2), R34.1
- net I2C_SCL: now reaches U1.35 (IO42)
- net I2C_SCL: now also J5.3 (Pin_3), R35.1
- net RX0: now reaches U1.36 (RXD0)
- net RX0: now also J2.3 (Pin_3), R79.2
- net TX0: now reaches U1.37 (TXD0)
- net TX0: now also J2.2 (Pin_2), R80.2
- net SP_SD: now reaches U1.38 (IO2)
- net SP_SD: now also J14.5 (Pin_5)
- net BUT1: now reaches U1.39 (IO1)
- net BUT1: now also C64.2, R44.2, SW3.1
- net RL2: now reaches U1.5 (IO5)
- net RL2: now also U6.2
- net RL3: now reaches U1.6 (IO6)
- net RL3: now also U7.2
- net IR_RX: now reaches U1.7 (IO7)
- net IR_RX: now also IC1.1 (OUT), R37.1
- net MIC_BCLK: now reaches U1.8 (IO15)
- net MIC_BCLK: now also J15.3 (Pin_3)
- net MIC_WS: now reaches U1.9 (IO16)
- net MIC_WS: now also J15.2 (Pin_2)
- removed net +3V3_ADS: C51.2, C52.2, C56.2
- removed net +5VD: C57.2, C58.2, R65.1, U22.3 (VI)
- removed net GNDA: R53.2, R54.2, R57.1, R58.1
- removed net GNDD: C51.1, C52.1, C56.1, C57.1, C58.1, C60.1, C61.1, C62.1, C63.1, C64.1, C65.1, U22.1 (GND)
- removed net VREFP: R52.1, R55.2, R56.2, R63.1, R64.1, R65.2
- new net: BL2.2 (IP), C71.2, R56.2
- new net: J14.4 (Pin_4), R41.2
- new net: D35.1 (K), R80.1
- new net: C51.1, IC1.3 (VS), R36.1
- new net: J9.B5 (CC2), R46.1
- new net: D34.1 (K), R79.1
- new net: BL1.2 (IP), C70.2, R53.2
- new net: D1.1 (K), Q1.3 (D)
- new net: D1.2 (A), R38.2
- new net: Q1.1 (G), R39.2, R40.1
- new net: D38.1 (K), R83.1
- new net: D33.1 (K), R78.1
- new net: J9.A5 (CC1), R45.1
- new net: J4.1 (Pin_1), R64.1
- new net: R63.2, TR1.1
- new net: J2.1 (Pin_1), R65.1
- new net: BL1.3 (IN), C69.1, R54.2
- new net: D36.1 (K), R81.1
- new net COM2: J12.2, K2.COM, R3.1
- new net COM3: J13.2, K3.COM, R4.1
- new net O2: C2.2, J12.1, K2.NO
- new net O3: C3.2, J13.1, K3.NO
- no-connect marks 7 -> 12
Other:
- note removed: "CONNECTOR"
- note removed: "IC ADS1256"
- note removed: "OP-AMP"
- note removed: "PWR - DECOUPLING"
- moved on the sheet: C57, C58, C60, C63, C65, D32, J1, J10, R77, U1, U22, U4

Commit message: done PCB
Parts:
- removed BL3: (no value), Package_SO:SSOP-10_3.9x4.9mm_P1.00mm, symbol Sym:BL0942
- removed C3: 47nF, Capacitor_THT:C_Disc_D10.5mm_W5.0mm_P7.50mm, symbol Device:C
- removed D10: LED, LED_SMD:LED_0805_2012Metric_Pad1.15x1.40mm_HandSolder, symbol Device:LED
- removed D14: SS34, Diode_SMD:D_SMA_Handsoldering, symbol Device:D
- removed J1, J11, J12, J13: KF7.62-2P, KF7.62:2P, symbol KF-7.62:KF7.62-2P
- removed J8: CT, Connector_JST:JST_XH_B2B-XH-A_1x02_P2.50mm_Vertical, symbol Connector:Conn_01x02_Pin
- removed K1, K2, K3: SRD-12VDC-SL-C, Footprint:RELAY_SRD-12VDC-SL-C, symbol RL10ASRD:SRD-12VDC-SL-C
- removed Q4: AO3400A, Package_TO_SOT_SMD:SOT-23, symbol Transistor_FET:AO3400A
- removed R27: 100, Resistor_SMD:R_0805_2012Metric_Pad1.20x1.40mm_HandSolder, symbol Device:R
- removed R28: 10K, Resistor_SMD:R_0805_2012Metric_Pad1.20x1.40mm_HandSolder, symbol Device:R
- removed R31: 4K1, Resistor_SMD:R_0805_2012Metric_Pad1.20x1.40mm_HandSolder, symbol Device:R
- removed R4: 100Ohm, Resistor_THT:R_Axial_DIN0414_L11.9mm_D4.5mm_P15.24mm_Horizontal, symbol Device:R
- removed R58, R62: 33R, Resistor_SMD:R_0805_2012Metric_Pad1.20x1.40mm_HandSolder, symbol Device:R
- removed R59, R60: 1K, Resistor_SMD:R_0805_2012Metric_Pad1.20x1.40mm_HandSolder, symbol Device:R
- removed R61, R63: 100K, Resistor_SMD:R_0805_2012Metric_Pad1.20x1.40mm_HandSolder, symbol Device:R
- removed TR1: ZMPT101K, Transformer_THT:Transformer_Zeming_ZMPT101K, symbol Transformer:ZMPT101K
- removed U22: AMS1117-3.3, Package_TO_SOT_SMD:SOT-223-3_TabPin2, symbol Regulator_Linear:AMS1117-3.3
- removed U4: HLK-5M05, Converter_ACDC:Converter_ACDC_Hi-Link_HLK-5Mxx, symbol Converter_ACDC:HLK-5M05
- removed U7: PC817, Footprint:SOP254P960X420-4N, symbol Isolator:PC817
- added 220-12V1: LS05_12V, Footprint:LS05-23BxxDR3, symbol Sym:LS05-23BxxDR3
- added AC_IN1, OUT1, OUT2: Conn_01x02_Pin, TerminalBlock_Phoenix:TerminalBlock_Phoenix_MKDS-1,5-2-5.08_1x02_P5.08mm_Horizontal, symbol Connector:Conn_01x02_Pin
- added C3: 10uF, Capacitor_SMD:CP_Elec_10x10.5, symbol Device:C_Polarized
- added C78, C79: 22uF, Resistor_SMD:R_0603_1608Metric_Pad0.98x0.95mm_HandSolder, symbol Device:C
- added IC2: TPS563200DDCR, Footprint:SOT95P280X110-6N, symbol Sym:TPS563200DDCR
- added K1, K2: Relay_SPDT, Relay_THT:Relay_SPDT_Schrack-RT1-16A-FormC_RM5mm, symbol Relay:Relay_SPDT
- added L1: 3.3uH, Inductor_SMD:L_7.3x7.3_H3.5, symbol Device:L
- added R82, R85: 10K, Resistor_SMD:R_0603_1608Metric_Pad0.98x0.95mm_HandSolder, symbol Device:R
- added R84: 54.9K, Resistor_SMD:R_0603_1608Metric_Pad0.98x0.95mm_HandSolder, symbol Device:R
- added U2: ME6211C50M5, Package_TO_SOT_SMD:SOT-23-5, symbol Regulator_Linear:ME6211C50M5
- C52, C56, C57, C58, C59, C60, C61, C62, C63, C64, C65, C66, C67, C69, C70, C71, C72, C73, R23, R24, R25, R26, R29, R30, R34, R35, R36, R37, R38, R39, R40, R41, R42, R43, R44, R52, R53, R54, R55, R56, R57, R64, R65, R72, R77, R78, R79, R80, R81, R83: footprint Resistor_SMD:R_0805_2012Metric_Pad1.20x1.40mm_HandSolder -> Resistor_SMD:R_0603_1608Metric_Pad0.98x0.95mm_HandSolder
- C74, C75: value 33nF -> 106; footprint Resistor_SMD:R_0805_2012Metric_Pad1.20x1.40mm_HandSolder -> Resistor_SMD:R_1206_3216Metric_Pad1.30x1.75mm_HandSolder
- C76: value 100uF -> 104; footprint Resistor_SMD:R_0805_2012Metric_Pad1.20x1.40mm_HandSolder -> Resistor_SMD:R_0603_1608Metric_Pad0.98x0.95mm_HandSolder
- C77: value 33nF -> 104; footprint Resistor_SMD:R_0805_2012Metric_Pad1.20x1.40mm_HandSolder -> Resistor_SMD:R_0603_1608Metric_Pad0.98x0.95mm_HandSolder
- J14: footprint Connector_PinHeader_1.00mm:PinHeader_1x07_P1.00mm_Vertical -> Connector_PinHeader_2.54mm:PinHeader_1x07_P2.54mm_Vertical
- J6: value CT -> CT1
- J7: value CT -> CT2
- R45, R46: footprint Resistor_SMD:R_0805_2012Metric -> Resistor_SMD:R_0603_1608Metric_Pad0.98x0.95mm_HandSolder
- U1: footprint RF_Module:ESP32-S3-WROOM-1 -> RF_Module:ESP32-S3-WROOM-1U
Connections:
- net +3V3: now also U2.5 (V_{OUT}); no longer C76.2
- net +5V: now also C78.1, C79.1, L1.2, R84.2, U2.1 (V_{IN}), U2.3 (CE); no longer D12.1 (K), D13.1 (K), D36.2 (A), U5.4, U6.4
- net BL_RX1: no longer BL2.10 (TX)
- net BL_RX2: now also BL2.10 (TX)
- net COM1: now also C1.2, K2.11, OUT1.2 (Pin_2); no longer R2.1
- net COM2: now also C2.2, K1.11, OUT2.2 (Pin_2); no longer R3.1
- net GND: now also C74.2, C76.2, 220-12V1.5 (-Vo), C78.2, C79.2, IC2.1 (GND), R85.1, U2.2 (V_{SS}); no longer C74.1, C76.1, C77.2
- net L: now also 220-12V1.1 (AC(L)), AC_IN1.1 (Pin_1)
- net N: now also 220-12V1.2 (AC(N)), AC_IN1.2 (Pin_2)
- net O1: now also R2.1, K2.14, OUT1.1 (Pin_1); no longer C1.2
- net O2: now also R3.1, K1.14, OUT2.1 (Pin_1); no longer C2.2
- net at D12.2 (A), Q2.3 (D): now also K2.A2
- net at D13.2 (A), Q3.3 (D): now also K1.A2
- net +12V: now reaches C75.1
- net +12V: now also C74.1, C76.1, D12.1 (K), D13.1 (K), D36.2 (A), U5.4, U6.4, 220-12V1.6 (+Vo), IC2.3 (VIN), K1.A1, K2.A1, R82.2
- net BL_RX3: no longer names the net of U1.20 (IO12)
- net RL3: no longer names the net of U1.6 (IO6)
- removed net VP: BL1.4 (VP), BL2.4 (VP), C77.1
- new net: IC2.4 (VFB), R84.1, R85.2
- new net: C77.2, IC2.2 (SW), L1.1
- new net: IC2.5 (EN), R82.1
- new net: C77.1, IC2.6 (VBST)
- new net: 220-12V1.3 (+V(cap)), C3.1
- new net: 220-12V1.4 (-V(cap)), C3.2
- no-connect marks 12 -> 15
Other:
- moved on the sheet: C1, C2, C56, C57, C58, C59, C60, C63, C65, D12, D13, J14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
