File: Hardware/PCB/IoT_Board/IoT_Board.kicad_sch (KiCad schematic)
At the start: 109 parts, among them IC1 VS1838B, IC2 TPS563200DDCR, J10 Conn_01x02_Pin, J14 MAX_98357, J15 INMP_441, J2 Debug UART0, J4 UART1, J5 I2C, J6 CT1, J7 CT2, J9 USB_C_Receptacle_USB2.0_16P, K1 Relay_SPDT, K2 Relay_SPDT, Q1 AO3400A, Q2 AO3400A, Q3 AO3400A, SW1 SW_Push, SW2 SW_Push, SW3 SW_Push, SW4 SW_Push, U1 ESP32-S3-WROOM-1, U2 ME6211C50M5, U5 PC817, U6 PC817

Commit message: Final
Parts:
- renumbered J10 to 5V1, J6 to CT1, J7 to CT2, J5 to I2C1, J15 to INMP_441, D8 to LED_RL1, D9 to LED_RL2, J14 to MAX_98357, J2 to UART0, J4 to UART1
Changed lines of the file:
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@@
 		(in_pos_files yes)
 		(dnp no)
-		(property "Reference" "J7"
+		(property "Reference" "CT2"
 			(at 304.546 191.262 0)
 			(show_name no)
@@
 			(project "IoT_Board"
 				(path "/f7f4c251-abef-4e4b-a993-341f87747a84"
-					(reference "J7")
+					(reference "CT2")
 					(unit 1)
 				)
@@
 		(dnp no)
 		(fields_autoplaced yes)
-		(property "Reference" "D9"
+		(property "Reference" "LED_RL2"
 			(at 279.7174 69.85 90)
 			(hide yes)
@@
 			(project "IoT_Board"
 				(path "/f7f4c251-abef-4e4b-a993-341f87747a84"
-					(reference "D9")
+					(reference "LED_RL2")
 					(unit 1)
 				)
@@
 		(dnp no)
 		(fields_autoplaced yes)
-		(property "Reference" "D8"
+		(property "Reference" "LED_RL1"
 			(at 279.7174 109.22 90)
 			(hide yes)
@@
 			(project "IoT_Board"
 				(path "/f7f4c251-abef-4e4b-a993-341f87747a84"
-					(reference "D8")
+					(reference "LED_RL1")
 					(unit 1)
 				)
@@
 		(in_pos_files yes)
 		(dnp no)
-		(property "Reference" "J6"
+		(property "Reference" "CT1"
 			(at 304.546 154.432 0)
 			(show_name no)
@@
 			(project "IoT_Board"
 				(path "/f7f4c251-abef-4e4b-a993-341f87747a84"
-					(reference "J6")
+					(reference "CT1")
 					(unit 1)
 				)
@@
 		(in_pos_files yes)
 		(dnp no)
-		(property "Reference" "J2"
+		(property "Reference" "UART0"
 			(at 31.242 34.29 90)
 			(show_name no)
@@
 			(project "IoT_Board"
 				(path "/f7f4c251-abef-4e4b-a993-341f87747a84"
-					(reference "J2")
+					(reference "UART0")
 					(unit 1)
 				)
@@
 		(dnp no)
 		(fields_autoplaced yes)
-		(property "Reference" "J15"
+		(property "Reference" "INMP_441"
 			(at 195.58 226.06 0)
 			(show_name no)
@@
 			(project "IoT_Board"
 				(path "/f7f4c251-abef-4e4b-a993-341f87747a84"
-					(reference "J15")
+					(reference "INMP_441")
 					(unit 1)
 				)
@@
 		(dnp no)
 		(fields_autoplaced yes)
-		(property "Reference" "J10"
+		(property "Reference" "5V1"
 			(at 169.545 264.16 0)
 			(show_name no)
@@
 			(project "IoT_Board"
 				(path "/f7f4c251-abef-4e4b-a993-341f87747a84"
-					(reference "J10")
+					(reference "5V1")
 					(unit 1)
 				)
@@
 		(in_pos_files yes)
 		(dnp no)
-		(property "Reference" "J5"
+		(property "Reference" "I2C1"
 			(at 31.242 76.708 90)
 			(show_name no)
@@
 			(project "IoT_Board"
 				(path "/f7f4c251-abef-4e4b-a993-341f87747a84"
-					(reference "J5")
+					(reference "I2C1")
 					(unit 1)
 				)
@@
 		(in_pos_files yes)
 		(dnp no)
-		(property "Reference" "J4"
+		(property "Reference" "UART1"
 			(at 31.496 53.34 90)
 			(show_name no)
@@
 			(project "IoT_Board"
 				(path "/f7f4c251-abef-4e4b-a993-341f87747a84"
-					(reference "J4")
+					(reference "UART1")
 					(unit 1)
 				)
@@
 		(dnp no)
 		(fields_autoplaced yes)
-		(property "Reference" "J14"
+		(property "Reference" "MAX_98357"
 			(at 186.055 198.12 0)
 			(show_name no)
@@
 			(project "IoT_Board"
 				(path "/f7f4c251-abef-4e4b-a993-341f87747a84"
-					(reference "J14")
+					(reference "MAX_98357")
 					(unit 1)
 				)

Commit message: add gerber OK
Parts:
- renumbered SW2 to BOOT, SW3 to BUT1, SW4 to BUT2, SW1 to EN
Changed lines of the file:
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@@
 		(dnp no)
 		(fields_autoplaced yes)
-		(property "Reference" "SW1"
+		(property "Reference" "EN"
 			(at 50.8 208.28 0)
 			(show_name no)
@@
 			(project "IoT_Board"
 				(path "/f7f4c251-abef-4e4b-a993-341f87747a84"
-					(reference "SW1")
+					(reference "EN")
 					(unit 1)
 				)
@@
 		(dnp no)
 		(fields_autoplaced yes)
-		(property "Reference" "SW4"
+		(property "Reference" "BUT2"
 			(at 50.8 250.19 0)
 			(show_name no)
@@
 			(project "IoT_Board"
 				(path "/f7f4c251-abef-4e4b-a993-341f87747a84"
-					(reference "SW4")
+					(reference "BUT2")
 					(unit 1)
 				)
@@
 		(dnp no)
 		(fields_autoplaced yes)
-		(property "Reference" "SW3"
+		(property "Reference" "BUT1"
 			(at 50.8 228.6 0)
 			(show_name no)
@@
 			(project "IoT_Board"
 				(path "/f7f4c251-abef-4e4b-a993-341f87747a84"
-					(reference "SW3")
+					(reference "BUT1")
 					(unit 1)
 				)
@@
 		(dnp no)
 		(fields_autoplaced yes)
-		(property "Reference" "SW2"
+		(property "Reference" "BOOT"
 			(at 52.07 186.69 0)
 			(show_name no)
@@
 			(project "IoT_Board"
 				(path "/f7f4c251-abef-4e4b-a993-341f87747a84"
-					(reference "SW2")
+					(reference "BOOT")
 					(unit 1)
 				)

Commit message: feat: Add Smart Home Gateway (Sherpa-ONNX, Qwen LLM, EdgeTTS, Closed-Loop Verifier), Master Plan & update PCB design
Parts:
- renumbered BOOT to BOOT1, EN to EN1
Changed lines of the file:
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@@
 		(dnp no)
 		(fields_autoplaced yes)
-		(property "Reference" "EN"
+		(property "Reference" "EN1"
 			(at 50.8 208.28 0)
 			(show_name no)
@@
 			(project "IoT_Board"
 				(path "/f7f4c251-abef-4e4b-a993-341f87747a84"
-					(reference "EN")
+					(reference "EN1")
 					(unit 1)
 				)
@@
 		(dnp no)
 		(fields_autoplaced yes)
-		(property "Reference" "BOOT"
+		(property "Reference" "BOOT1"
 			(at 52.07 186.69 0)
 			(show_name no)
@@
 			(project "IoT_Board"
 				(path "/f7f4c251-abef-4e4b-a993-341f87747a84"
-					(reference "BOOT")
+					(reference "BOOT1")
 					(unit 1)
 				)

Commit message: firmware
Connections:
- net BL_RX2: no longer BL2.6 (CF1)
- no-connect marks 15 -> 17
Changed lines of the file:
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@@
+	)
+	(no_connect
+		(at 387.35 201.93)
 	)
 	(no_connect
@@
 	(no_connect
 		(at 114.3 59.69)
+	)
+	(no_connect
+		(at 387.35 165.1)
 	)
 	(no_connect
@@
 			)
 			(justify left bottom)
-		)
-	)
-	(label "BL_RX2"
-		(at 387.35 201.93 0)
-		(effects
-			(font
-				(size 1.27 1.27)
-				(thickness 0.1588)
-			)
-			(justify left bottom)

Commit message: fix nhieu bug
Changed lines of the file:
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@@
 	(wire
 		(pts
-			(xy 204.47 240.03) (xy 204.47 237.49)
-		)
-		(stroke
-			(width 0)
-			(type default)
-		)
-	)
-	(wire
-		(pts
 			(xy 74.93 44.45) (xy 83.82 44.45)
 		)
@@
 	(wire
 		(pts
-			(xy 204.47 237.49) (xy 201.93 237.49)
+			(xy 203.2 237.49) (xy 201.93 237.49)
 		)
 		(stroke
@@
 	)
 	(label "MIC_DIN"
-		(at 204.47 240.03 0)
+		(at 203.2 237.49 0)
 		(effects
 			(font
@@
 		)
 		(property "Value" "+3V3"
-			(at 205.74 236.474 90)
+			(at 211.074 234.95 90)
 			(show_name no)
 			(do_not_autoplace no)
@@
 		(in_pos_files yes)
 		(dnp no)
-		(fields_autoplaced yes)
 		(property "Reference" "INMP_441"
-			(at 195.58 226.06 0)
+			(at 180.086 228.6 0)
 			(show_name no)
 			(do_not_autoplace no)

Commit message: push 1.10
Parts:
- C3: value 10uF -> 400V 10uF
Changed lines of the file:
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@@
 			)
 		)
-		(property "Value" "10uF"
+		(property "Value" "400V 10uF"
 			(at 207.518 282.956 0)
 			(show_name no)
