File: Hardware/PCB/IoT_Board/_restore_backup_2026-09-03T19-50-40-326/IoT_Board.kicad_pcb (KiCad board)
At the start: 2 copper layers, 100 x 50 mm, 109 parts, among them IC1 VS1838B, IC2 TPS563200DDCR, J10 Conn_01x02_Pin, J14 MAX_98357, J15 INMP_441, J2 Debug UART0, J4 UART1, J5 I2C, J6 CT1, J7 CT2, J9 USB_C_Receptacle_USB2.0_16P, K1 Relay_SPDT, K2 Relay_SPDT, Q1 AO3400A, Q2 AO3400A, Q3 AO3400A, SW1 SW_Push, SW2 SW_Push, SW3 SW_Push, SW4 SW_Push, U1 ESP32-S3-WROOM-1, U2 ME6211C50M5, U5 PC817, U6 PC817

Commit message: OK
Parts:
- R23, R24: value 220 -> 100
- V G SD R DO BLK LRC: renamed from J14
- renumbered J2 to ., J4 to ., SW2 to BOOT, SW1 to EN
Connections:
- R23 pad 1: +5V -> +3V3
- R24 pad 1: +5V -> +3V3
Routing:
- net +5V: track 166.7 -> 119.9 mm, vias 4 -> 3
- net +3V3: track 116.9 -> 121.1 mm
Changed lines of the file:
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@@
 		(descr "Tactile switch, SPST, 6.0x3.5 mm, H2.5 mm, straight, NO, gull wing leads: https://www.ckswitches.com/media/2779/pts636.pdf")
 		(tags "switch tactile SPST 1P1T straight NO SMTR C&K")
-		(property "Reference" "SW1"
+		(property "Reference" "EN"
 			(at -4.325 -1.6 0)
 			(unlocked yes)
@@
 		(descr "JST XH series connector, B4B-XH-A (http://www.jst-mfg.com/product/pdf/eng/eXH.pdf)")
 		(tags "connector JST XH vertical")
-		(property "Reference" "J2"
+		(property "Reference" "."
 			(at -0.05 -2.9 0)
 			(layer "F.SilkS")
@@
 			(unit
 				(name "A")
-				(pins "SH" "B1" "B12" "A1" "A12" "A9" "B4" "B9" "A4" "A5" "B5" "A7" "B7"
+				(pins "SH" "A1" "A12" "B1" "B12" "A4" "A9" "B4" "B9" "A5" "B5" "A7" "B7"
 					"A6" "B6" "A8" "B8"
 				)
@@
 		(sheetname "/")
 		(sheetfile "IoT_Board.kicad_sch")
-		(units
-			(unit
-				(name "A")
-				(pins "3" "27" "39" "38" "15" "4" "5" "6" "7" "12" "17" "18" "19" "20"
-					"21" "22" "8" "9" "2" "41" "40" "1" "37" "36" "10" "11" "13" "14" "23"
-					"28" "29" "30" "31" "32" "33" "34" "35" "26" "16" "24" "25"
-				)
-			)
-		)
 		(attr smd)
 		(duplicate_pad_numbers_are_jumpers no)
@@
 		(descr "Through hole straight pin header, 1x07, 2.54mm pitch, single row")
 		(tags "Through hole pin header THT 1x07 2.54mm single row")
-		(property "Reference" "J14"
+		(property "Reference" "V G SD R DO BLK LRC"
 			(at 2.4 8.045 180)
 			(layer "F.SilkS")
@@
 		(descr "Tactile switch, SPST, 6.0x3.5 mm, H2.5 mm, straight, NO, gull wing leads: https://www.ckswitches.com/media/2779/pts636.pdf")
 		(tags "switch tactile SPST 1P1T straight NO SMTR C&K")
-		(property "Reference" "SW2"
+		(property "Reference" "BOOT"
 			(at -8.1 -0.05 0)
 			(unlocked yes)
@@
 		(descr "JST XH series connector, B4B-XH-A (http://www.jst-mfg.com/product/pdf/eng/eXH.pdf)")
 		(tags "connector JST XH vertical")
-		(property "Reference" "J4"
+		(property "Reference" "."
 			(at -0.025 3.725 0)
 			(layer "F.SilkS")
@@
 		(sheetname "/")
 		(sheetfile "IoT_Board.kicad_sch")
-		(units
-			(unit
-				(name "A")
-				(pins "1" "2" "3" "4" "6" "5")
-			)
-		)
 		(duplicate_pad_numbers_are_jumpers no)
 		(fp_line
@@
 			)
 		)
-		(property "Value" "220"
+		(property "Value" "100"
 			(at 0 -1.43 0)
 			(layer "B.Fab")
@@
 			(layers "B.Cu" "B.Mask" "B.Paste")
 			(roundrect_rratio 0.25)
-			(net "+5V")
+			(net "+3V3")
 			(pintype "passive")
 		)
@@
 			)
 		)
-		(property "Value" "220"
+		(property "Value" "100"
 			(at 0 -1.43 0)
 			(layer "B.Fab")
@@
 			(layers "B.Cu" "B.Mask" "B.Paste")
 			(roundrect_rratio 0.25)
-			(net "+5V")
+			(net "+3V3")
 			(pintype "passive")
 		)
@@
 	)
 	(segment
+		(start 77.4875 183.2)
+		(end 75.65 185.0375)
+		(width 0.3)
+		(layer "B.Cu")
+		(net "+3V3")
+	)
+	(segment
 		(start 96.75 166.2)
 		(end 91.3 171.65)
@@
 	)
 	(segment
+		(start 77.4875 181.6)
+		(end 77.4875 183.2)
+		(width 0.3)
+		(layer "B.Cu")
+		(net "+3V3")
+	)
+	(segment
 		(start 63.9 151.229167)
 		(end 63.183333 150.5125)
@@
 	)
 	(segment
-		(start 73.600001 171.155454)
-		(end 66.955455 177.8)
-		(width 0.3)
-		(layer "F.Cu")
-		(net "+5V")
-	)
-	(segment
 		(start 96.675 145.9)
 		(end 96.35 146.225)
@@
 	)
 	(segment
-		(start 65.975 161.275)
-		(end 67.275 161.275)
-		(width 0.3)
-		(layer "F.Cu")
-		(net "+5V")
-	)
-	(segment
-		(start 66.955455 177.8)
-		(end 66.2 177.8)
-		(width 0.3)
-		(layer "F.Cu")
-		(net "+5V")
-	)
-	(segment
 		(start 63.05 157.65)
 		(end 63.607108 157.092892)
@@
 	)
 	(segment
-		(start 65.362432 157.65)
-		(end 65.975 158.262568)
-		(width 0.3)
-		(layer "F.Cu")
-		(net "+5V")
-	)
-	(segment
-		(start 75.6 182.35)
-		(end 76.1 181.85)
-		(width 0.3)
-		(layer "F.Cu")
-		(net "+5V")
-	)
-	(segment
 		(start 109.0125 147.525)
 		(end 108.8375 147.7)
@@
 	)
 	(segment
-		(start 66.2 180.5)
-		(end 68.05 182.35)
-		(width 0.3)
-		(layer "F.Cu")
-		(net "+5V")
-	)
-	(segment
 		(start 108.475 144.3)
 		(end 108.075 143.9)
@@
 	)
 	(segment
-		(start 66.2 177.8)
-		(end 66.2 180.5)
-		(width 0.3)
-		(layer "F.Cu")
-		(net "+5V")
-	)
-	(segment
-		(start 73.600001 167.600001)
-		(end 73.600001 171.155454)
-		(width 0.3)
-		(layer "F.Cu")
-		(net "+5V")
-	)
-	(segment
 		(start 108.8375 147.7)
 		(end 108.8375 149.35)
@@
 	)
 	(segment
-		(start 67.275 161.275)
-		(end 73.600001 167.600001)
-		(width 0.3)
-		(layer "F.Cu")
-		(net "+5V")
-	)
-	(segment
 		(start 104.25 146.325)
 		(end 105.3 145.275)
@@
 	)
 	(segment
-		(start 63.05 157.65)
-		(end 65.362432 157.65)
-		(width 0.3)
-		(layer "F.Cu")
-		(net "+5V")
-	)
-	(segment
 		(start 106.7 145.275)
 		(end 108.1 143.875)
@@
 	)
 	(segment
-		(start 68.05 182.35)
-		(end 75.6 182.35)
-		(width 0.3)
-		(layer "F.Cu")
-		(net "+5V")
-	)
-	(segment
 		(start 77.88 161.3)
 		(end 77.93 161.25)
@@
 	)
 	(segment
-		(start 65.975 158.262568)
-		(end 65.975 161.275)
-		(width 0.3)
-		(layer "F.Cu")
-		(net "+5V")
-	)
-	(segment
 		(start 60.95 141.725)
 		(end 61.725 140.95)
@@
 	)
 	(via
-		(at 76.1 181.85)
-		(size 0.6)
-		(drill 0.3)
-		(layers "F.Cu" "B.Cu")
-		(net "+5V")
-	)
-	(via
 		(at 99.45 140.975)
 		(size 0.6)
@@
 	)
 	(segment
-		(start 77.4875 183.2)
-		(end 77.4875 181.6)
-		(width 0.3)
-		(layer "B.Cu")
-		(net "+5V")
-	)
-	(segment
-		(start 76.35 181.6)
-		(end 76.1 181.85)
-		(width 0.3)
-		(layer "B.Cu")
-		(net "+5V")
-	)
-	(segment
 		(start 108.175 142.6875)
 		(end 108.1 142.7625)
 		(width 0.3)
 		(layer "B.Cu")
-		(net "+5V")
-	)
-	(segment
-		(start 77.4875 181.6)
-		(end 76.35 181.6)
-		(width 0.3)
-		(layer "B.Cu")
