File: Hardware/PCB/IoT_Board/_restore_backup_2026-09-03T19-50-40-326/IoT_Board.kicad_sch (KiCad schematic)
At the start: 109 parts, among them IC1 VS1838B, IC2 TPS563200DDCR, J10 Conn_01x02_Pin, J14 MAX_98357, J15 INMP_441, J2 Debug UART0, J4 UART1, J5 I2C, J6 CT1, J7 CT2, J9 USB_C_Receptacle_USB2.0_16P, K1 Relay_SPDT, K2 Relay_SPDT, Q1 AO3400A, Q2 AO3400A, Q3 AO3400A, SW1 SW_Push, SW2 SW_Push, SW3 SW_Push, SW4 SW_Push, U1 ESP32-S3-WROOM-1, U2 ME6211C50M5, U5 PC817, U6 PC817

Commit message: OK
Parts:
- R23, R24: value 220 -> 100
Changed lines of the file:
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@@
 			)
 		)
-		(property "Value" "220"
+		(property "Value" "100"
 			(at 271.78 69.85 90)
 			(show_name no)
@@
 			)
 		)
-		(property "Value" "220"
+		(property "Value" "100"
 			(at 271.78 109.22 90)
 			(show_name no)
